Commit message: Add electronics box, RP Lidar cylinder and Realsense 435 box

File: robco_4wd_mecanum_description/urdf/left_wheel_assy_macros.xacro (robot description, xacro)
@@ -1,4 +1,57 @@
 <?xml version="1.0"?>
 <robot xmlns:xacro="http://www.ros.org/wiki/xacro">
+  <xacro:macro name="fixed_joint" params="name parent_name child_name color *origin">
+  <joint name="${name}_link_joint" type="fixed">
+    <parent link="${parent_name}"/>
+    <child link="${child_name}"/>
+    <insert_block name="origin" />
+  </joint>
+  </xacro:macro>
+  <xacro:macro name="box_link" params="name lenght width height mass color *origin">
+  <link name="${name}_link">
+    <visual>
+    <!-- The chassis is represented with a box and the origin of that box is in it's center.
+    That's why, in order to visualize properly, we need to add half of the box height to
+    the distance from the ground allready defined in the joint. -->
+      <origin xyz="0 0 ${height/2}" rpy="0 0 0" />
+      <geometry>
+        <!-- <mesh filename="package://robco_4wd_mecanum_description/meshes/robco_base_link.STL" scale="0.001 0.001 0.001"/> -->
+        <box size="${lenght} ${width} ${height}"/>
+      </geometry>
+      <!-- <material name="light_grey" /> -->
+      <material name="${color}" />
+    </visual>
+    <collision>
+      <origin xyz="0 0 0" rpy="0 0 0" />
+      <geometry>
+        <box size="${lenght} ${width} ${height}"/>
+      </geometry>
+    </collision>
+    <!-- Ivoke box_inertial_with_origin macro -->
+    <xacro:box_inertial_with_origin x="${lenght}" y="${width}" z="${height}" mass="${mass}">
+      <origin xyz="0 0 0" rpy="0 0 0" />
+    </xacro:box_inertial_with_origin>
+  </link>
+  </xacro:macro>
+  <xacro:macro name="cylinder_link" params="name radius lenght mass color *origin">
+  <link name="${name}_link">
+    <visual>
+      <insert_block name="origin" />
+      <geometry>
+        <cylinder radius="${radius}" length="${lenght}"/>
+      </geometry>
+      <material name="${color}" />
+    </visual>
+    <collision>
+      <insert_block name="origin" />
+      <geometry>
+        <cylinder radius="${radius}" length="${lenght}"/>
+      </geometry>
+    </collision>
+    <xacro:cylinder_inertial_with_origin radius="${radius}" length="${lenght}" mass="${mass}">
+      <insert_block name="origin" />
+    </xacro:cylinder_inertial_with_origin>
+  </link>
+  </xacro:macro>
   <xacro:macro name="shaft_joint" params="name *origin">
   <joint name="${name}_wheel_shaft_joint" type="fixed">

File: robco_4wd_mecanum_description/urdf/robco_4wd_mecanum.xacro (robot description, xacro)
@@ -81,5 +81,5 @@
     <xacro:property name="chassis_height" value="${89*SCALE_mm_to_m}" />
     <xacro:property name="chassis_half_height" value="${chassis_height/2}" />  <!-- 34.5 *SCALE_mm_to_m-->
-    <xacro:property name="chassis_weight" value="${19.0-4*0.7}" /> <!-- in kg-->
+    <xacro:property name="chassis_mass" value="${19.0-4*0.7}" /> <!-- in kg-->
     <!-- Chassis: distance from the ground to bottom -->
     <xacro:property name="chassis_bottom_z_offset" value="${40.2*SCALE_mm_to_m}" />
@@ -148,24 +148,19 @@
       <geometry>
         <!-- <mesh filename="package://robco_4wd_mecanum_description/meshes/robco_base_link.STL" scale="0.001 0.001 0.001"/> -->
-      <box size="${chassis_lenght} ${chassis_width} ${chassis_height}"/>
+        <box size="${chassis_lenght} ${chassis_width} ${chassis_height}"/>
       </geometry>
       <!-- <material name="light_grey" /> -->
-      <material name="White" />
+      <material name="Orange" />
     </visual>
     <collision>
-      <origin xyz="0 0 0"/>
+      <origin xyz="0 0 0" rpy="0 0 0" />
       <geometry>
         <box size="${chassis_lenght} ${chassis_width} ${chassis_height}"/>
       </geometry>
     </collision>
-    <inertial>
-      <!-- Inertia from CAD model, filled box assumption -->
-      <origin xyz="-0.01103 0 0.002" rpy="0 0 0"/>
-      <mass value="2.844"/>
-      <inertia
-        ixx="0.018819942" ixy="0" ixz="-0.000101519"
-        iyy="0.057333716" iyz="0"
-        izz="0.074201740"/>
-    </inertial>
+    <!-- Ivoke box_inertial_with_origin macro -->
+    <xacro:box_inertial_with_origin x="${chassis_lenght}" y="${chassis_width}" z="${chassis_height}" mass="${chassis_mass}">
+      <origin xyz="0 0 0" rpy="0 0 0" />
+    </xacro:box_inertial_with_origin>
   </link>
   <joint name="front_left_wheel_shaft_joint" type="fixed">
@@ -202,5 +197,6 @@
     <axis xyz="0 1 0"/>
   </joint>
-  <!-- <link name="front_left_wheel">
+<!-- Wheel link version with cylinders   -->
+  <!-- <link name="front_left_wheel_link">
     <visual>
       <origin xyz="0 ${wheel_width/2} 0" rpy="${ROTATE_90_DEGREES} 0 0" />
@@ -226,4 +222,5 @@
     </inertial>
   </link>  -->
+<!-- Wheel link version with mesh   -->
   <link name="front_left_wheel_link">
     <visual>
@@ -303,4 +300,64 @@
       <origin xyz="0 ${-shaft_lenght} 0" rpy="0 0 0" />
     </xacro:wheel_link>
+<!-- **** ELECTRONICS BOX (MODULE) - height 100 mm ****  -->
+<!-- /batteries height is 76 mm whenlaying on the side. -->
+<!-- can accomadete, not only Raspberry PI 4 with passive cooling case,  -->
+<!-- but also  Intel NUC in the big case 51 mm height/ -->
+<!-- ! The Joint is positioned on top plane of the chassis (base_link) module -->
+  <xacro:fixed_joint name="electronics_box" parent_name="base_link" child_name="electronics_box_link" color="Grey">
+    <origin xyz="0 0 ${chassis_height}" rpy="0 0 0" />
+  </xacro:fixed_joint>
+  <xacro:box_link name="electronics_box" lenght="${chassis_lenght}" width="${chassis_width}" height="${100*SCALE_mm_to_m}" mass="15" color="yellow">
+    <origin xyz="0 0 ${100*SCALE_mm_to_m/2}" rpy="0 0 0" />
+  </xacro:box_link>
+<!-- **** ROBOT TORSO STANDOFF (POLE) height = 406.8 mm ****  -->
+<!-- The heap is located at about 0.53 of the human body lenght -->
+<!-- Robot haight - 1200 mm, Heap height from the ground = 1200 mm * 0.53 = 636 mm -->
+<!-- Torso standoff height is 636 mm - base_plate_botom_from_base_frame_Z_offset - chassis_height - electronics_box_height  -->
+<!-- standoff_height = 636 - 40.2 - 89 - 100 = 406.8 -->
+<!-- aluminium profile 40x40 will be used weight of the profile is: 2.45 kg/meter -->
+<!-- ! The Joint is positioned on top plane of the electronics box module -->
+  <xacro:fixed_joint name="torso_standoff" parent_name="electronics_box_link" child_name="torso_standoff_link" color="Grey">
+    <origin xyz="0 0 ${100*SCALE_mm_to_m}" rpy="0 0 0" />
+  </xacro:fixed_joint>
+  <xacro:box_link name="torso_standoff" lenght="${40*SCALE_mm_to_m}" width="${40*SCALE_mm_to_m}" height="${406.8*SCALE_mm_to_m}" mass="${2.45*0.4068}" color="Blue">
+    <origin xyz="0 0 ${406.8*SCALE_mm_to_m/2}" rpy="0 0 0" />
+  </xacro:box_link>
+<!--  **** RP LIDAR A2 **** -->
+<!-- Position the RP Lidar 10 mm from the front edge of the electronics box, to avoid the chance of collision, just in case. -->
+<!-- RP Lidar's /diameter 75.7 mm/ center point needs to be at x = (337.5 - 10) - (75.7/2) = 289.65 mm from the box center -->
+<!-- ! The Joint is positioned on top plane of the electronics box module -->
+  <xacro:fixed_joint name="rplidar" parent_name="electronics_box_link" child_name="rplidar_link" color="Red">
+    <origin xyz="${289.65*SCALE_mm_to_m} 0 ${100*SCALE_mm_to_m}" rpy="0 0 0" />
+  </xacro:fixed_joint>
+  <!-- <xacro:box_link name="rplidar" lenght="0.01" width="0.01" height="0.01" mass="0.01" color="Orange">
+    <origin xyz="0 0 0" rpy="0 0 0" />
+  </xacro:box_link> -->
+  <xacro:cylinder_link name="rplidar" radius="${75.7/2*SCALE_mm_to_m}" lenght="${40.80*SCALE_mm_to_m}" mass="${0.190}" color="Orange">
+    <origin xyz="0 0 ${40.80/2*SCALE_mm_to_m}" rpy="0 0 0" />
+ </xacro:cylinder_link>
+<!-- **** Intel RealSense Depth Camera D435 ****  -->
+<!-- dimensions 90 mm × 25 mm × 25 mm    weight 258.5477 g. -->
+<!-- ! The Joint is positioned on the front plane of the torso standoff at height of ?? -->
+  <xacro:fixed_joint name="realsense" parent_name="electronics_box_link" child_name="realsense_link" color="Red">
+    <origin xyz="${(20)*SCALE_mm_to_m} 0 ${(100+350)*SCALE_mm_to_m}" rpy="0 1.8326 0" />
+  </xacro:fixed_joint>
+  <xacro:box_link name="realsense" lenght="${25*SCALE_mm_to_m}" width="${90*SCALE_mm_to_m}" height="${25*SCALE_mm_to_m}" mass="0.2585477" color="Orange">
+    <origin xyz="0 0 0" rpy="0 0 0" />
+  </xacro:box_link>
+<!-- Camera direction VISUALIZER -->
+  <!-- <xacro:fixed_joint name="module_visualizer" parent_name="realsense_link" child_name="realsense_visualizer_link" color="Red">
+    <origin xyz="0 0 0" rpy="0 0 0" />
+  </xacro:fixed_joint>
+  <xacro:box_link name="realsense_visualizer" lenght="0.01" width="0.01" height="0.1" mass="0.01" color="Red">
+       <origin xyz="0 0 0" rpy="0 0 0" />
+  </xacro:box_link> -->
+<!-- JOINT AND LINK VISUALIZERS -->
+  <!-- <xacro:fixed_joint name="module_visualizer" parent_name="base_link" child_name="module_visualizer_link" color="Red">
+    <origin xyz="0 0 0.5" rpy="0 0 0" />
+  </xacro:fixed_joint>
+  <xacro:box_link name="module_visualizer" lenght="0.05" width="0.05" height="0.05" mass="0.01" color="Red">
+       <origin xyz="0 0 0" rpy="0 0 0" />
+  </xacro:box_link> -->
   <!-- Include URM04 ultrasonic range finders -->
   <!-- <xacro:include filename="$(find robco_4wd_mecanum_description)/urdf/urm04_sensor.xacro"/> -->

Commit message: Add RP Lidar A2 and ORBBEC Astra with meshes

File: robco_4wd_mecanum_description/urdf/left_wheel_assy_macros.xacro (robot description, xacro)
@@ -1,9 +1,9 @@
 <?xml version="1.0"?>
-<robot xmlns:xacro="http://www.ros.org/wiki/xacro">
+<robot xmlns:xacro="http://ros.org/wiki/xacro">
   <xacro:macro name="fixed_joint" params="name parent_name child_name color *origin">
   <joint name="${name}_link_joint" type="fixed">
     <parent link="${parent_name}"/>
     <child link="${child_name}"/>
-    <insert_block name="origin" />
+    <xacro:insert_block name="origin" />
   </joint>
   </xacro:macro>
@@ -37,5 +37,5 @@
   <link name="${name}_link">
     <visual>
-      <insert_block name="origin" />
+      <xacro:insert_block name="origin" />
       <geometry>
         <cylinder radius="${radius}" length="${lenght}"/>
@@ -44,5 +44,5 @@
     </visual>
     <collision>
-      <insert_block name="origin" />
+      <xacro:insert_block name="origin" />
       <geometry>
         <cylinder radius="${radius}" length="${lenght}"/>
@@ -50,5 +50,5 @@
     </collision>
     <xacro:cylinder_inertial_with_origin radius="${radius}" length="${lenght}" mass="${mass}">
-      <insert_block name="origin" />
+      <xacro:insert_block name="origin" />
     </xacro:cylinder_inertial_with_origin>
   </link>
@@ -58,5 +58,5 @@
     <parent link="base_link"/>
     <child link="${name}_wheel_shaft_link" />
-    <insert_block name="origin" />
+    <xacro:insert_block name="origin" />
   </joint>
   </xacro:macro>
@@ -64,5 +64,5 @@
   <link name="${name}_wheel_shaft_link">
     <visual>
-      <insert_block name="origin" />
+      <xacro:insert_block name="origin" />
       <geometry>
         <cylinder radius="${radius}" length="${lenght}"/>
@@ -71,5 +71,5 @@
     </visual>
     <collision>
-      <insert_block name="origin" />
+      <xacro:insert_block name="origin" />
       <geometry>
         <cylinder radius="${radius}" length="${lenght}"/>
@@ -77,5 +77,5 @@
     </collision>
     <xacro:cylinder_inertial_with_origin radius="${radius}" length="${lenght}" mass="${mass}">
-      <insert_block name="origin" />
+      <xacro:insert_block name="origin" />
     </xacro:cylinder_inertial_with_origin>
   </link>
@@ -83,8 +83,8 @@
   <xacro:macro name="wheel_joint" params="name *origin *axis">
   <joint name="${name}_wheel_joint" type="fixed">
-    <insert_block name="origin" />
+    <xacro:insert_block name="origin" />
     <parent link="${name}_wheel_shaft_link"/>
     <child link="${name}_wheel_link" />
-    <insert_block name="axis" />
+    <xacro:insert_block name="axis" />
   </joint>
   </xacro:macro>
@@ -92,5 +92,5 @@
   <link name="${name}_wheel_link">
     <visual>
-    <insert_block name="origin" />
+    <xacro:insert_block name="origin" />
       <geometry>
         <mesh filename="${mesh_file_name}" scale="${mesh_scale_x} ${mesh_scale_y} ${mesh_scale_z}"/>
@@ -99,5 +99,5 @@
     </visual>
     <collision>
-    <insert_block name="origin" />
+    <xacro:insert_block name="origin" />
       <geometry>
         <cylinder radius="${radius}" length="${width}"/>
@@ -105,6 +105,37 @@
     </collision>
     <xacro:cylinder_inertial_with_origin radius="${radius}" length="${width}" mass="${mass}">
-    <insert_block name="origin" />
+    <xacro:insert_block name="origin" />
     </xacro:cylinder_inertial_with_origin>
+  </link>
+  </xacro:macro>
+  <!-- **** RP LIDAR A2 **** -->
+  <!-- SHOULD Z ROTATE THE LIDAR JOINT 180 !!!  -->
+  <!-- <joint name="rplidar_joint" type="fixed">
+    <axis xyz="0 1 0" />
+    <origin xyz="0.02 0 0.058" rpy="0 0 3.14"/>
+    <parent link="base_link"/>
+    <child link="laser"/>
+  </joint> -->
+    <!-- ! USE THIS ORIGIN TO ALLIGN THE DAE VISUAL: -->
+    <!-- <origin xyz="0 0 0" rpy="1.5707 0 4.71"/> -->
+  <xacro:macro name="rplidar_a2" params="name *origin">
+  <link name="${name}_link">
+    <visual>
+    <xacro:insert_block name="origin" />
+      <geometry>
+        <mesh filename="package://robco_4wd_mecanum_description/meshes/rplidar.dae" scale="0.001 0.001 0.001"/>
+      </geometry>
+    </visual>
+    <collision>
+    <xacro:insert_block name="origin" />
+      <geometry>
+        <mesh filename="package://robco_4wd_mecanum_description/meshes/rplidar.dae" scale="0.001 0.001 0.001"/>
+      </geometry>
+    </collision>
+    <inertial>
+      <mass value="1e-5" />
+      <xacro:insert_block name="origin" />
+      <inertia ixx="0" ixy="0" ixz="0" iyy="0" iyz="0" izz="0" />
+    </inertial>
   </link>
   </xacro:macro>

File: robco_4wd_mecanum_description/urdf/robco_4wd_mecanum.xacro (robot description, xacro)
@@ -227,5 +227,5 @@
       <origin xyz="0 ${shaft_lenght} 0" rpy="0 0 0"/>
       <geometry>
-        <mesh filename="package://nexus_4wd_mecanum_description/meshes/mecanum_wheel_left.STL" scale="${1*SCALE_mm_to_m} ${0.92*SCALE_mm_to_m} ${1.52*SCALE_mm_to_m}"/>
+        <mesh filename="package://robco_4wd_mecanum_description/meshes/mecanum_wheel_left.STL" scale="${1*SCALE_mm_to_m} ${0.92*SCALE_mm_to_m} ${1.52*SCALE_mm_to_m}"/>
       </geometry>
       <material name="light_grey"/>
@@ -274,5 +274,5 @@
 <!-- Invoke wheel_joint macros for the back left wheel -->
     <xacro:wheel_link name="back_left" radius="${wheel_radius}" width="${wheel_width}" mass="${wheel_mass}" color="light_grey"
-      mesh_file_name="package://nexus_4wd_mecanum_description/meshes/mecanum_wheel_left.STL" mesh_scale_x="${1*SCALE_mm_to_m}"
+      mesh_file_name="package://robco_4wd_mecanum_description/meshes/mecanum_wheel_left.STL" mesh_scale_x="${1*SCALE_mm_to_m}"
       mesh_scale_y="${0.92*SCALE_mm_to_m}" mesh_scale_z="${1.52*SCALE_mm_to_m}">
       <origin xyz="0 ${shaft_lenght} 0" rpy="0 0 0" />
@@ -285,5 +285,5 @@
 <!-- Invoke wheel_joint macros for the front right wheel -->
     <xacro:wheel_link name="front_right" radius="${wheel_radius}" width="${wheel_width}" mass="${wheel_mass}" color="light_grey"
-      mesh_file_name="package://nexus_4wd_mecanum_description/meshes/mecanum_wheel_right.STL" mesh_scale_x="${1*SCALE_mm_to_m}"
+      mesh_file_name="package://robco_4wd_mecanum_description/meshes/mecanum_wheel_right.STL" mesh_scale_x="${1*SCALE_mm_to_m}"
       mesh_scale_y="${0.92*SCALE_mm_to_m}" mesh_scale_z="${1.52*SCALE_mm_to_m}">
       <origin xyz="0 ${-shaft_lenght} 0" rpy="0 0 0" />
@@ -296,5 +296,5 @@
 <!-- Invoke wheel_joint macros for the back right wheel -->
     <xacro:wheel_link name="back_right" radius="${wheel_radius}" width="${wheel_width}" mass="${wheel_mass}" color="light_grey"
-      mesh_file_name="package://nexus_4wd_mecanum_description/meshes/mecanum_wheel_right.STL" mesh_scale_x="${1*SCALE_mm_to_m}"
+      mesh_file_name="package://robco_4wd_mecanum_description/meshes/mecanum_wheel_right.STL" mesh_scale_x="${1*SCALE_mm_to_m}"
       mesh_scale_y="${0.92*SCALE_mm_to_m}" mesh_scale_z="${1.52*SCALE_mm_to_m}">
       <origin xyz="0 ${-shaft_lenght} 0" rpy="0 0 0" />
@@ -328,22 +328,102 @@
 <!-- RP Lidar's /diameter 75.7 mm/ center point needs to be at x = (337.5 - 10) - (75.7/2) = 289.65 mm from the box center -->
 <!-- ! The Joint is positioned on top plane of the electronics box module -->
-  <xacro:fixed_joint name="rplidar" parent_name="electronics_box_link" child_name="rplidar_link" color="Red">
+  <!-- **** RP LIDAR A2 CYLINDER VISUALISATION -->
+  <!-- <xacro:fixed_joint name="rplidar" parent_name="electronics_box_link" child_name="rplidar_link" color="Red">
     <origin xyz="${289.65*SCALE_mm_to_m} 0 ${100*SCALE_mm_to_m}" rpy="0 0 0" />
-  </xacro:fixed_joint>
+  </xacro:fixed_joint> -->
+   <!-- RP Lidar A2 cylinder visual -->
+  <!-- <xacro:cylinder_link name="rplidar" radius="${75.7/2*SCALE_mm_to_m}" lenght="${40.80*SCALE_mm_to_m}" mass="${0.190}" color="Orange">
+    <origin xyz="0 0 ${40.80/2*SCALE_mm_to_m}" rpy="0 0 0" />
+  </xacro:cylinder_link> -->
+  <!-- Mount point (joint) visual marker -->
   <!-- <xacro:box_link name="rplidar" lenght="0.01" width="0.01" height="0.01" mass="0.01" color="Orange">
     <origin xyz="0 0 0" rpy="0 0 0" />
   </xacro:box_link> -->
-  <xacro:cylinder_link name="rplidar" radius="${75.7/2*SCALE_mm_to_m}" lenght="${40.80*SCALE_mm_to_m}" mass="${0.190}" color="Orange">
-    <origin xyz="0 0 ${40.80/2*SCALE_mm_to_m}" rpy="0 0 0" />
- </xacro:cylinder_link>
+  <!-- <xacro:fixed_joint name="rplidar" parent_name="electronics_box_link" child_name="rplidar_link" color="Grey">
+    <origin xyz="${289.65*SCALE_mm_to_m} 0 ${100*SCALE_mm_to_m}" rpy="0 0 3.14" />
+  </xacro:fixed_joint> -->
+  <!-- <xacro:rplidar_a2 name="rplidar">
+    <origin xyz="0 0 0" rpy="1.5707 0 4.71"/>
+  </xacro:rplidar_a2> -->
+<joint name="rplidar_joint" type="fixed">
+    <axis xyz="0 1 0" />
+    <origin xyz="${289.65*SCALE_mm_to_m} 0 ${100*SCALE_mm_to_m}" rpy="0 0 3.14" />
+    <parent link="electronics_box_link"/>
+    <child link="laser"/>
+  </joint>
+  <!-- rplidar Laser -->
+  <link name="laser">
+    <visual>
+      <origin xyz="0 0 0" rpy="1.5707 0 4.71"/>
+      <geometry>
+        <mesh filename="package://robco_4wd_mecanum_description/meshes/rplidar.dae" scale="0.001 0.001 0.001"/>
+      </geometry>
+    </visual>
+    <collision>
+      <origin xyz="0 0 0" rpy="1.5707 0 4.71"/>
+      <geometry>
+        <mesh filename="package://robco_4wd_mecanum_description/meshes/rplidar.dae" scale="0.001 0.001 0.001"/>
+      </geometry>
+    </collision>
+    <inertial>
+      <mass value="1e-5" />
+      <origin xyz="0 0 0" rpy="1.5707 0 4.71"/>
+      <inertia ixx="0" ixy="0" ixz="0" iyy="0" iyz="0" izz="0" />
+    </inertial>
+  </link>
+<!-- **** ORBBEC ASTRA Depth Camera  ****  -->
+  <!-- Orbbec Astra RGBD Camera -->
+  <joint name="astra_joint" type="fixed">
+    <!-- <axis xyz="0 0 0" /> -->
+    <!-- <origin xyz="-0.03 0 0.18" rpy="0 0 0"/> -->
+    <origin xyz="${(75)*SCALE_mm_to_m} 0 ${(100+350)*SCALE_mm_to_m}" rpy="0 0.261799 0" />
+    <!-- <origin xyz="${(20)*SCALE_mm_to_m} 0 ${(100+350)*SCALE_mm_to_m}" rpy="0 1.8326 0" /> -->
+    <parent link="electronics_box_link"/>
+    <child link="camera_link"/>
+  </joint>
+  <link name="camera_link">
+    <collision>
+      <origin xyz="0.02 0 0" rpy="0 0 0"/>
+      <geometry>0
+        <box size="0.001 0.001 0.001"/>
+      </geometry>
+    </collision>
+    <visual>
+      <origin xyz="-0.01 0 -0.03" rpy="1.5707 0 1.5707"/>
+      <geometry>
+        <mesh filename="package://robco_4wd_mecanum_description/meshes/astra.dae" scale="0.001 0.001 0.001" />
+      </geometry>
+    </visual>
+    <inertial>
+      <mass value="1e-5" />
+      <origin xyz="0 0 0" rpy="0 0 0"/>
+      <inertia ixx="0" ixy="0" ixz="0" iyy="0" iyz="0" izz="0" />
+    </inertial>
+  </link>
+  <joint name="camera_optical_joint" type="fixed">
+    <origin xyz="0 0 0" rpy="${-pi/2} 0 ${-pi/2}"/>
+    <parent link="camera_link"/>
+    <child link="camera_rgb_frame"/>
+  </joint>
+  <link name="camera_rgb_frame">
+  </link>
+  <joint name="camera_depth_joint" type="fixed">
+    <origin xyz="0 0 0" rpy="${-pi/2} 0 ${-pi/2}"/>
+    <parent link="camera_link"/>
+    <child link="camera_depth_frame"/>
+  </joint>
+  <link name="camera_depth_frame">
+  </link>
+  <!-- ******************** =============================== ************************************ -->
 <!-- **** Intel RealSense Depth Camera D435 ****  -->
 <!-- dimensions 90 mm × 25 mm × 25 mm    weight 258.5477 g. -->
 <!-- ! The Joint is positioned on the front plane of the torso standoff at height of ?? -->
-  <xacro:fixed_joint name="realsense" parent_name="electronics_box_link" child_name="realsense_link" color="Red">
+  <!-- <xacro:fixed_joint name="realsense" parent_name="electronics_box_link" child_name="realsense_link" color="Red">
     <origin xyz="${(20)*SCALE_mm_to_m} 0 ${(100+350)*SCALE_mm_to_m}" rpy="0 1.8326 0" />
   </xacro:fixed_joint>
   <xacro:box_link name="realsense" lenght="${25*SCALE_mm_to_m}" width="${90*SCALE_mm_to_m}" height="${25*SCALE_mm_to_m}" mass="0.2585477" color="Orange">
     <origin xyz="0 0 0" rpy="0 0 0" />
-  </xacro:box_link>
+  </xacro:box_link> -->
+<!-- JOINT AND LINK VISUALIZERS -->
 <!-- Camera direction VISUALIZER -->
   <!-- <xacro:fixed_joint name="module_visualizer" parent_name="realsense_link" child_name="realsense_visualizer_link" color="Red">
@@ -353,5 +433,4 @@
        <origin xyz="0 0 0" rpy="0 0 0" />
   </xacro:box_link> -->
-<!-- JOINT AND LINK VISUALIZERS -->
   <!-- <xacro:fixed_joint name="module_visualizer" parent_name="base_link" child_name="module_visualizer_link" color="Red">
     <origin xyz="0 0 0.5" rpy="0 0 0" />
