Commit message: Remove non ascii unicode character

File: robco_4wd_mecanum_description/urdf/left_wheel_assy_macros.xacro (robot description, xacro)
@@ -119,4 +119,5 @@
     <!-- ! USE THIS ORIGIN TO ALLIGN THE DAE VISUAL: -->
     <!-- <origin xyz="0 0 0" rpy="1.5707 0 4.71"/> -->
+<!--
   <xacro:macro name="rplidar_a2" params="name *origin">
   <link name="${name}_link">
@@ -139,5 +140,5 @@
     </inertial>
   </link>
-  </xacro:macro>
+  </xacro:macro>     -->
 </robot>
   <!-- <link name="${name}">

File: robco_4wd_mecanum_description/urdf/robco_4wd_mecanum.xacro (robot description, xacro)
@@ -372,11 +372,9 @@
     </inertial>
   </link>
-<!-- **** ORBBEC ASTRA Depth Camera  ****  -->
-  <!-- Orbbec Astra RGBD Camera -->
+<!-- **** ORBBEC ASTRA RGBD CAMERA  ****  -->
   <joint name="astra_joint" type="fixed">
-    <!-- <axis xyz="0 0 0" /> -->
-    <!-- <origin xyz="-0.03 0 0.18" rpy="0 0 0"/> -->
+    <axis xyz="0 0 0" />
+    <!-- <origin xyz="${(20)*SCALE_mm_to_m} 0 ${(100+350)*SCALE_mm_to_m}" rpy="0 1.8326 0" /> -->
     <origin xyz="${(75)*SCALE_mm_to_m} 0 ${(100+350)*SCALE_mm_to_m}" rpy="0 0.261799 0" />
-    <!-- <origin xyz="${(20)*SCALE_mm_to_m} 0 ${(100+350)*SCALE_mm_to_m}" rpy="0 1.8326 0" /> -->
     <parent link="electronics_box_link"/>
     <child link="camera_link"/>
@@ -417,5 +415,5 @@
   <!-- ******************** =============================== ************************************ -->
 <!-- **** Intel RealSense Depth Camera D435 ****  -->
-<!-- dimensions 90 mm × 25 mm × 25 mm    weight 258.5477 g. -->
+<!-- dimensions 90 mm x 25 mm x 25 mm    weight 258.5477 g. -->
 <!-- ! The Joint is positioned on the front plane of the torso standoff at height of ?? -->
   <!-- <xacro:fixed_joint name="realsense" parent_name="electronics_box_link" child_name="realsense_link" color="Red">
